File: jbeacon/jbeacon.kicad_pcb (KiCad board)
At the start: 2 copper layers, 25.7 x 35 mm, 12 parts, among them J1 PROGRAMMING_POGO, Y1 Crystal_26MHz

Commit message: more cleanup
Other:
- board text added: "TODO: confirm IC footprint 50ohm antenna trace impedance"
- board text removed: "TODO: confirm IC footprint 50ohm antenna trace impedance finalize dimensions"
Changed lines of the file:
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@@
 		(layer "Dwgs.User")
-	)
-	(gr_circle
-		(center 105 105)
-		(end 110 105)
-		(stroke
-			(width 0.1)
-			(type default)
-		)
-		(fill none)
-		(layer "Cmts.User")
 	)
 	(gr_arc
@@
 		(layer "Edge.Cuts")
 	)
-	(gr_text "TODO:\nconfirm IC footprint\n50ohm antenna trace impedance\nfinalize dimensions"
+	(gr_text "TODO:\nconfirm IC footprint\n50ohm antenna trace impedance"
 		(at 127.85 123.95 0)
 		(layer "Cmts.User")

Commit message: case CAD
Parts:
- H1: renamed from REF**; value MountingHole_3mm -> KEYCHAIN_HOLE
- Y1: footprint Crystal:Crystal_SMD_SeikoEpson_FA128-4Pin_2.0x1.6mm -> project:OSC_XRCGB26M000F2P00R0
- moved Y1 0.35 mm to (122.4, 122.2), turned to -90 degrees
- moved AE1 0.16 mm to (120.3, 134.7)
