File: jbeacon/jbeacon.kicad_sch (KiCad schematic)
At the start: 11 parts, among them J1 PROGRAMMING_POGO, Y1 Crystal_26MHz

Commit message: case CAD
Parts:
- added H1: KEYCHAIN_HOLE, MountingHole:MountingHole_3mm, symbol Mechanical:MountingHole
- Y1: footprint Crystal:Crystal_SMD_SeikoEpson_FA128-4Pin_2.0x1.6mm -> project:OSC_XRCGB26M000F2P00R0
Changed lines of the file:
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@@
 			)
 		)
-		(property "Footprint" "Crystal:Crystal_SMD_SeikoEpson_FA128-4Pin_2.0x1.6mm"
+		(property "Footprint" "project:OSC_XRCGB26M000F2P00R0"
 			(at 101.6 111.76 0)
 			(effects
@@
 					(unit 1)
 				)
+			)
+		)
+	)
+	(symbol
+		(lib_id "Mechanical:MountingHole")
+		(at 220.98 78.74 0)
+		(unit 1)
+		(exclude_from_sim yes)
+		(in_bom no)
+		(on_board yes)
+		(dnp no)
+		(fields_autoplaced yes)
+		(property "Reference" "H1"
+			(at 223.52 77.4699 0)
+			(effects
+				(font
+					(size 1.27 1.27)
+				)
+				(justify left)
+			)
+		)
+		(property "Value" "KEYCHAIN_HOLE"
+			(at 223.52 80.0099 0)
+			(effects
+				(font
+					(size 1.27 1.27)
+				)
+				(justify left)
+			)
+		)
+		(property "Footprint" "MountingHole:MountingHole_3mm"
+			(at 220.98 78.74 0)
+			(effects
+				(font
+					(size 1.27 1.27)
+				)
+				(hide yes)
+			)
+		)
+		(property "Datasheet" "~"
+			(at 220.98 78.74 0)
+			(effects
+				(font
+					(size 1.27 1.27)
+				)
+				(hide yes)
+			)
+		)
+		(property "Description" "Mounting Hole without connection"
+			(at 220.98 78.74 0)
+			(effects
+				(font
+					(size 1.27 1.27)
+				)
+				(hide yes)
+			)
+		)
+		(instances
+			(project ""
+				(path "/654510c1-a06c-4e16-9820-d5980f5e3c7b"
+					(reference "H1")
+					(unit 1)
+				)
